Commit message: diffbot.urdf 작게

File: src/my_map/models/diffbot.urdf (robot description, URDF)
Before this commit: robot diffbot, 6 links, 5 joints
Links:
- link base_link: geometry visual box size=0.2 0.1 0.05
- link left_wheel_link: geometry visual cylinder length=0.02 radius=0.025
- link right_wheel_link: geometry visual cylinder length=0.02 radius=0.025
Joints:
- joint camera_joint: origin xyz=0.15 0 0.12 rpy=0 0 0 -> xyz=0.1 0 0.08 rpy=0 0 0
- joint caster_joint: origin xyz=-0.15 0 0.015 rpy=0 0 0 -> xyz=-0.08 0 0.025 rpy=0 0 0
- joint left_wheel_joint: origin xyz=0.1 0.1 0.05 rpy=0 0 0 -> xyz=0.05 0.06 0.025 rpy=0 0 0
- joint lidar_joint: origin xyz=0 0 0.17 rpy=0 0 0 -> xyz=0 0 0.1 rpy=0 0 0
- joint right_wheel_joint: origin xyz=0.1 -0.1 0.05 rpy=0 0 0 -> xyz=0.05 -0.06 0.025 rpy=0 0 0
